File: Geist.kicad_sch (KiCad schematic)
At the start: 46 parts, among them J1 USB_C_Receptacle_USB2.0_16P, J2 Conn_01x05, J3 Conn_01x03, J4 Conn_01x07, J5 Conn_01x05, J6 Conn_01x02, J7 Conn_01x02, J8 Conn_01x02, J9 Conn_01x02, U1 LM27762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

Commit message: GND pour
laid gnd pour on the pcb and adjusted some pins to suit better routing. Will work on chopping down DRC next.
Connections:
- net BUTTON_NEXT: now also U3.23 (IO21); no longer U3.10 (IO17)
- net BUTTON_PLAY: now also U3.22 (IO14); no longer U3.9 (IO16)
- net BUTTON_PREV: now also U3.21 (IO13); no longer U3.8 (IO15)
- net I2S_BCLK: now also U3.27 (IO0); no longer U3.23 (IO21)
- net KNOB_A: now also U3.38 (IO2); no longer U3.4 (IO4)
- net KNOB_B: now also U3.35 (IO42); no longer U3.5 (IO5)
- net KNOB_SW: now also U3.34 (IO41); no longer U3.6 (IO6)
- net TFT_CS: now also U3.4 (IO4); no longer U3.18 (IO10)
- net TOGGLE_MODE: now also U3.33 (IO40); no longer U3.7 (IO7)
Changed lines of the file:
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@@
 	)
 	(no_connect
-		(at 99.06 166.37)
+		(at 68.58 163.83)
 	)
 	(no_connect
@@
 	)
 	(no_connect
-		(at 99.06 176.53)
+		(at 68.58 153.67)
 	)
 	(no_connect
-		(at 99.06 168.91)
+		(at 68.58 179.07)
 	)
 	(no_connect
@@
 	)
 	(no_connect
-		(at 68.58 171.45)
+		(at 68.58 156.21)
 	)
 	(no_connect
@@
 	)
 	(no_connect
-		(at 68.58 173.99)
-	)
-	(no_connect
-		(at 68.58 143.51)
-	)
-	(no_connect
-		(at 99.06 163.83)
+		(at 68.58 151.13)
 	)
 	(no_connect
@@
 	)
 	(no_connect
+		(at 99.06 176.53)
+	)
+	(no_connect
 		(at 99.06 158.75)
 	)
 	(no_connect
-		(at 68.58 138.43)
+		(at 99.06 138.43)
 	)
 	(no_connect
@@
 		(at 99.06 156.21)
 	)
+	(no_connect
+		(at 68.58 176.53)
+	)
 	(wire
 		(pts
@@
 			(width 0)
 			(type default)
+		)
+	)
+	(label "KNOB_A"
+		(at 68.58 143.51 180)
+		(effects
+			(font
+				(size 1.27 1.27)
+			)
+			(justify right bottom)
 		)
 	)
@@
 		)
 	)
+	(label "I2S_BCLK"
+		(at 68.58 138.43 180)
+		(effects
+			(font
+				(size 1.27 1.27)
+			)
+			(justify right bottom)
+		)
+	)
 	(label "I2S_LRCK"
 		(at 99.06 151.13 0)
@@
 		)
 	)
+	(label "BUTTON_PLAY"
+		(at 68.58 173.99 180)
+		(effects
+			(font
+				(size 1.27 1.27)
+			)
+			(justify right bottom)
+		)
+	)
 	(label "TFT_SCLK"
 		(at 68.58 168.91 180)
@@
 		)
 	)
-	(label "TFT_CS"
-		(at 68.58 163.83 180)
-		(effects
-			(font
-				(size 1.27 1.27)
-			)
-			(justify right bottom)
-		)
-	)
 	(label "I2S_BCLK"
 		(at 158.75 113.03 180)
@@
 		)
 	)
-	(label "BUTTON_PLAY"
-		(at 68.58 179.07 180)
-		(effects
-			(font
-				(size 1.27 1.27)
-			)
-			(justify right bottom)
-		)
-	)
 	(label "OUT_L+"
 		(at 237.49 97.79 90)
@@
 		)
 	)
+	(label "TOGGLE_MODE"
+		(at 99.06 163.83 0)
+		(effects
+			(font
+				(size 1.27 1.27)
+			)
+			(justify left bottom)
+		)
+	)
 	(label "KNOB_SW"
 		(at 144.78 181.61 180)
@@
 		)
 	)
-	(label "BUTTON_PREV"
-		(at 68.58 176.53 180)
-		(effects
-			(font
-				(size 1.27 1.27)
-			)
-			(justify right bottom)
-		)
-	)
 	(label "TFT_CS"
 		(at 124.46 179.07 180)
@@
 		)
 	)
+	(label "KNOB_B"
+		(at 99.06 168.91 0)
+		(effects
+			(font
+				(size 1.27 1.27)
+			)
+			(justify left bottom)
+		)
+	)
+	(label "TFT_CS"
+		(at 68.58 148.59 180)
+		(effects
+			(font
+				(size 1.27 1.27)
+			)
+			(justify right bottom)
+		)
+	)
 	(label "+4.5V_Audio"
 		(at 107.95 26.67 0)
@@
 		)
 	)
+	(label "BUTTON_NEXT"
+		(at 99.06 148.59 0)
+		(effects
+			(font
+				(size 1.27 1.27)
+			)
+			(justify left bottom)
+		)
+	)
 	(label "3.3V"
 		(at 45.72 128.27 0)
@@
 		)
 	)
+	(label "KNOB_SW"
+		(at 99.06 166.37 0)
+		(effects
+			(font
+				(size 1.27 1.27)
+			)
+			(justify left bottom)
+		)
+	)
 	(label "USB_D+"
 		(at 45.72 53.34 0)
@@
 		)
 	)
-	(label "I2S_BCLK"
-		(at 99.06 148.59 0)
-		(effects
-			(font
-				(size 1.27 1.27)
-			)
-			(justify left bottom)
-		)
-	)
 	(label "TFT_RST"
 		(at 124.46 173.99 180)
@@
 		)
 	)
-	(label "KNOB_SW"
-		(at 68.58 153.67 180)
-		(effects
-			(font
-				(size 1.27 1.27)
-			)
-			(justify right bottom)
-		)
-	)
-	(label "KNOB_B"
-		(at 68.58 151.13 180)
-		(effects
-			(font
-				(size 1.27 1.27)
-			)
-			(justify right bottom)
-		)
-	)
 	(label "XSMT"
 		(at 99.06 140.97 0)
@@
 		)
 	)
+	(label "BUTTON_PREV"
+		(at 68.58 171.45 180)
+		(effects
+			(font
+				(size 1.27 1.27)
+			)
+			(justify right bottom)
+		)
+	)
 	(label "OUT_R+"
 		(at 217.17 58.42 0)
@@
 		)
 	)
-	(label "KNOB_A"
-		(at 68.58 148.59 180)
-		(effects
-			(font
-				(size 1.27 1.27)
-			)
-			(justify right bottom)
-		)
-	)
-	(label "TOGGLE_MODE"
-		(at 68.58 156.21 180)
-		(effects
-			(font
-				(size 1.27 1.27)
-			)
-			(justify right bottom)
-		)
-	)
 	(label "BUTTON_PREV"
 		(at 156.21 157.48 90)
@@
 		(effects
 			(font
-				(size 1.27 1.27)
-			)
-			(justify left bottom)
-		)
-	)
-	(label "BUTTON_NEXT"
-		(at 99.06 138.43 0)
-		(effects
-			(font

Commit message: PCB Finished
FIxed all DRCs and made further design decisions like making usb c connector hang 1mm off the edge. Added mounting holes. PCB finished. Will add bitmap in next commit.
Connections:
- net +4.5V_Audio: no longer U5.4 (V-)
- net -4.5V_Audio: now also U5.4 (V-)
Changed lines of the file:
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@@
+	)
+	(junction
+		(at 156.21 54.61)
+		(diameter 0)
+		(color 0 0 0 0)
 	)
 	(junction
@@
 	)
 	(junction
-		(at 160.02 26.67)
-		(diameter 0)
-		(color 0 0 0 0)
-	)
-	(junction
 		(at 153.67 163.83)
 		(diameter 0)
@@
 	)
 	(junction
-		(at 160.02 45.72)
-		(diameter 0)
-		(color 0 0 0 0)
-	)
-	(junction
 		(at 154.94 125.73)
 		(diameter 0)
@@
 	)
 	(junction
-		(at 160.02 54.61)
-		(diameter 0)
-		(color 0 0 0 0)
-	)
-	(junction
 		(at 134.62 76.2)
 		(diameter 0)
@@
 	)
 	(junction
+		(at 152.4 46.99)
+		(diameter 0)
+		(color 0 0 0 0)
+	)
+	(junction
 		(at 171.45 137.16)
 		(diameter 0)
@@
 	(junction
 		(at 101.6 184.15)
+		(diameter 0)
+		(color 0 0 0 0)
+	)
+	(junction
+		(at 156.21 26.67)
 		(diameter 0)
 		(color 0 0 0 0)
@@
 	(wire
 		(pts
-			(xy 160.02 54.61) (xy 166.37 54.61)
-		)
-		(stroke
-			(width 0)
-			(type default)
-		)
-	)
-	(wire
-		(pts
 			(xy 69.85 121.92) (xy 109.22 121.92)
 		)
@@
 	(wire
 		(pts
-			(xy 146.05 54.61) (xy 160.02 54.61)
+			(xy 146.05 54.61) (xy 156.21 54.61)
 		)
 		(stroke
@@
 	(wire
 		(pts
+			(xy 152.4 45.72) (xy 166.37 45.72)
+		)
+		(stroke
+			(width 0)
+			(type default)
+		)
+	)
+	(wire
+		(pts
 			(xy 41.91 128.27) (xy 46.99 128.27)
 		)
@@
 	(wire
 		(pts
-			(xy 160.02 26.67) (xy 166.37 26.67)
+			(xy 146.05 26.67) (xy 156.21 26.67)
 		)
 		(stroke
@@
 	(wire
 		(pts
+			(xy 156.21 26.67) (xy 156.21 54.61)
+		)
+		(stroke
+			(width 0)
+			(type default)
+		)
+	)
+	(wire
+		(pts
 			(xy 134.62 120.65) (xy 158.75 120.65)
 		)
@@
 	(wire
 		(pts
+			(xy 152.4 45.72) (xy 152.4 46.99)
+		)
+		(stroke
+			(width 0)
+			(type default)
+		)
+	)
+	(wire
+		(pts
 			(xy 115.57 73.66) (xy 121.92 73.66)
 		)
@@
 	(wire
 		(pts
-			(xy 160.02 45.72) (xy 166.37 45.72)
-		)
-		(stroke
-			(width 0)
-			(type default)
-		)
-	)
-	(wire
-		(pts
 			(xy 173.99 102.87) (xy 173.99 100.33)
 		)
@@
 	(wire
 		(pts
-			(xy 160.02 26.67) (xy 160.02 45.72)
-		)
-		(stroke
-			(width 0)
-			(type default)
-		)
-	)
-	(wire
-		(pts
 			(xy 21.59 128.27) (xy 26.67 128.27)
 		)
@@
 	(wire
 		(pts
-			(xy 146.05 26.67) (xy 160.02 26.67)
-		)
-		(stroke
-			(width 0)
-			(type default)
-		)
-	)
-	(wire
-		(pts
 			(xy 241.3 106.68) (xy 241.3 111.76)
 		)
@@
 	(wire
 		(pts
-			(xy 160.02 45.72) (xy 160.02 54.61)
-		)
-		(stroke
-			(width 0)
-			(type default)
-		)
-	)
-	(wire
-		(pts
 			(xy 106.68 73.66) (xy 113.03 73.66)
 		)
@@
 	(wire
 		(pts
+			(xy 156.21 26.67) (xy 166.37 26.67)
+		)
+		(stroke
+			(width 0)
+			(type default)
+		)
+	)
+	(wire
+		(pts
 			(xy 242.57 105.41) (xy 242.57 124.46)
 		)
@@
 		)
 		(stroke
+			(width 0)
+			(type default)
+		)
+	)
+	(wire
+		(pts
+			(xy 156.21 54.61) (xy 166.37 54.61)
+		)
+		(stroke
